File: EC65/jayec65/jay_EC65.kicad_pcb (KiCad board)
At the start: 2 copper layers, 300 x 100.8 mm, 169 parts, among them J1 USB_C_Receptacle_USB2.0, J2 USB_C_Receptacle_USB2.0, J3 JST, J4 Conn_01x04_Socket, J5 Conn_01x04_Socket, SW1 EC_SW, SW10 EC_SW, SW11 EC_SW, SW12 EC_SW, SW13 EC_SW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

Commit message: add
Parts:
- removed U10, U8: LTC6255IS6TRMPBF_flipped_power, Package_TO_SOT_SMD:TSOT-23-6_HandSoldering
- removed U7, U9: 74HC4051, cipulot_parts:TSSOP16
Routing:
- net GND: track 300.0 -> 316.2 mm, vias 33 -> 34
- net C1: track 193.2 -> 205.3 mm, vias 0 -> 1
