File: EC65/jayec65/jay_EC65.kicad_sch (KiCad schematic)
At the start: 37 parts, among them J1 USB_C_Receptacle_USB2.0, J2 USB_C_Receptacle_USB2.0, J3 JST, J4 Conn_01x04_Socket, J5 Conn_01x04_Socket, U1 STM32F401CBUx, U10 LTC6255IS6TRMPBF_flipped_power, U5 XC6206PxxxMR, U6 SRV05-4, U7 74HC4051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

Commit message: add
Parts:
- removed U10, U8: LTC6255IS6TRMPBF_flipped_power, Package_TO_SOT_SMD:TSOT-23-6_HandSoldering, symbol cipulot_parts:LTC6255IS6TRMPBF_flipped_power
- removed U7, U9: 74HC4051, cipulot_parts:TSSOP16, symbol 74xx:74HC4051
